Commit message: Changes to Camera Visuals

File: laika_description/urdf/camera.xacro (robot description, xacro)
@@ -5,6 +5,5 @@
         <visual>
             <geometry>
-                <!--cylinder radius="0.005" length="0.003"/-->
-                <box size="0.005 0.005 0.005"/>
+                <sphere radius="0.005" length="0.003"/>
             </geometry>
             <material name="white"/>
@@ -14,5 +13,5 @@
         <parent link="base_link"/>
         <child link="camera_link"/>
-        <origin xyz="0.146 0 0.076" rpy="0 0 0"/>
+        <origin xyz="0.144 0 0.076" rpy="0 0 0"/>
     </joint>
     <joint name="camera_optical_joint" type="fixed">

Commit message: Camera visibility and motor controller addition

File: laika_description/urdf/camera.xacro (robot description, xacro)
@@ -5,5 +5,5 @@
         <visual>
             <geometry>
-                <cylinder radius="0.005" length="0.003"/>
+                <sphere radius="0.005" length="0.003"/>
             </geometry>
             <material name="white"/>
@@ -13,5 +13,5 @@
         <parent link="base_link"/>
         <child link="camera_link"/>
-        <origin xyz="0.146 0 0.076" rpy="0 0 0"/>
+        <origin xyz="0.144 0 0.076" rpy="0 0 0"/>
     </joint>
     <joint name="camera_optical_joint" type="fixed">
