Commit message: More ros2_control amends

File: src/laika_description/urdf/sim.xacro (robot description, xacro)
@@ -106,5 +106,5 @@
                 <plugin>gazebo_ros2_control/GazeboSystem</plugin>
             </hardware>
-            <joint name="left_wheel_joint">
+            <joint name="base_to_left_front_wheel">
                 <command_interface name="velocity">
                     <param name="min">-10</param>
@@ -114,5 +114,5 @@
                 <state_interface name="position"/>
             </joint>
-            <joint name="right_wheel_joint">
+            <joint name="base_to_right_front_wheel">
                 <command_interface name="velocity">
                     <param name="min">-10</param>
@@ -125,9 +125,9 @@
     <gazebo>
         <plugin name="gazebo_ros2_control" filename="libgazebo_ros2_control.so">
-            <parameters>$(find laika_description)/config/my_controllers.yaml</parameters>
-            <parameters>$(find laika_description)/config/gaz_ros2_ctl_use_sim.yaml</parameters>
+            <parameters>$(find laika_description)/my_controllers.yaml</parameters>
+            <parameters>$(find laika_description)/gaz_ros2_ctl_use_sim.yaml</parameters>
         </plugin>
     </gazebo>
-<!-- Joint State Publisher and Pose -->
+<!-- Joint State Publisher and Pose
     <gazebo>
       <plugin name="gazebo_ros_joint_state_publisher"
@@ -139,5 +139,5 @@
         <joint_name>base_to_left_back_wheel</joint_name>
       </plugin>
-    </gazebo>
+    </gazebo -->
     <!--Note:  In startup the following error will occur:
     "[rviz2-5] Warning: Invalid frame ID "left_back_wheel" passed to canTransform argument source_frame - frame does not exist"

Commit message: Completed Simulator

File: src/laika_description/urdf/sim.xacro (robot description, xacro)
@@ -122,25 +122,25 @@
                 <state_interface name="position"/>
             </joint>
+            <joint name="base_to_left_back_wheel">
+                <command_interface name="velocity">
+                    <param name="min">-10</param>
+                    <param name="max">10</param>
+                </command_interface>
+                <state_interface name="velocity"/>
+                <state_interface name="position"/>
+            </joint>
+            <joint name="base_to_right_back_wheel">
+                <command_interface name="velocity">
+                    <param name="min">-10</param>
+                    <param name="max">10</param>
+                </command_interface>
+                <state_interface name="velocity"/>
+                <state_interface name="position"/>
+            </joint>
         </ros2_control>
     <gazebo>
         <plugin name="gazebo_ros2_control" filename="libgazebo_ros2_control.so">
-            <parameters>$(find laika_description)/my_controllers.yaml</parameters>
-            <parameters>$(find laika_description)/gaz_ros2_ctl_use_sim.yaml</parameters>
+            <parameters>$(find laika_description)/gazebo_controllers.yaml</parameters>
         </plugin>
     </gazebo>
-<!-- Joint State Publisher and Pose
-    <gazebo>
-      <plugin name="gazebo_ros_joint_state_publisher"
-          filename="libgazebo_ros_joint_state_publisher.so">
-        <update_rate>20</update_rate>
-        <joint_name>base_to_right_front_wheel</joint_name>
-        <joint_name>base_to_left_front_wheel</joint_name>
-        <joint_name>base_to_right_back_wheel</joint_name>
-        <joint_name>base_to_left_back_wheel</joint_name>
-      </plugin>
-    </gazebo -->
-    <!--Note:  In startup the following error will occur:
-    "[rviz2-5] Warning: Invalid frame ID "left_back_wheel" passed to canTransform argument source_frame - frame does not exist"
-    This will disappear when the Gazebo Joint State Publisher is running.
-     -->
 </robot>
